Commit message: add color to robot body

File: catkin_ws/src/my_robot/urdf/my_robot.xacro (robot description, xacro)
@@ -56,4 +56,7 @@
     </visual>
   </link>
+  <gazebo reference="chassis">
+    <material>Gazebo/Blue</material>
+  </gazebo>
   <link name="left_wheel">
 	<collision name='left_wheel_collision'>
